File: Power_US_Driver/Power_US_Driver.sch (KiCad schematic (older format))
At the start: 2 parts, among them J1 Conn_01x03, J2 Conn_Coaxial

Commit message: moved high current diode off board
Parts:
- J1: symbol Conn_01x03 -> Conn_01x05
Connections:
- net Power_Supply/HOT renamed Power_Supply/hot-240
- net Power_Supply/Nuetral renamed Power_Supply/neutral-240
- new net Power_Supply/Nuetral-120: J1.4 (Pin_4)
- new net Power_Supply/hot-120v: J1.5 (Pin_5)
Other:
- note added: "check for dumb shit w/ pwr, gnd. don't kill people"
- note added: "coax sheath is connected to case gnd"
- note added: "external voltage boost xformer may be applied for high voltage stage"
- note added: "reactification for 240 supply is off board."
- note added: "substantially reduces board space if large reactifier off board"
Changed lines of the file:
@@
 F1 "Power_Supply.sch" 60
 F2 "V+" O R 3350 2700 60
-F3 "HOT" I L 2300 2550 60
-F4 "Nuetral" I L 2300 2650 60
-F5 "12v" O R 3350 3300 60
-F6 "3v3" O R 3350 3600 60
+F3 "hot-120v" I L 2300 2550 60
+F4 "Nuetral-120" I L 2300 2650 60
+F5 "5v" O R 3350 3600 60
+F6 "hot-240" I L 2300 2750 60
+F7 "neutral-240" I L 2300 2850 60
 $EndSheet
 $Sheet
@@
 F0 "phase_comp" 60
 F1 "phase_comp.sch" 60
-F2 "US_SIG" I L 5350 5000 60
-F3 "PWR_OUT" O R 6350 5000 60
+F2 "PWR_OUT" O R 6350 5000 60
+F3 "PWR_IN" I L 5350 5000 60
+F4 "5v" I L 5350 5300 60
+F5 "Viout" O R 6350 5350 60
+F6 "Vsense" O R 6350 5200 60
 $EndSheet
 $Comp
-L Conn_01x03 J1
+L Conn_01x05 J1
 U 1 1 5AAE7F4F
-P 1900 2650
-F 0 "J1" H 1900 2850 50  0000 C CNN
-F 1 "Conn_01x03" H 1900 2450 50  0000 C CNN
-F 2 "" H 1900 2650 50  0001 C CNN
-F 3 "" H 1900 2650 50  0001 C CNN
-	1    1900 2650
+P 1750 2750
+F 0 "J1" H 1750 2950 50  0000 C CNN
+F 1 "Conn_01x03" H 1750 2450 50  0000 C CNN
+F 2 "" H 1750 2750 50  0001 C CNN
+F 3 "" H 1750 2750 50  0001 C CNN
+	1    1750 2750
 	-1   0    0    1
 $EndComp
@@
 	3650 4750 3850 4750
 Wire Wire Line
-	2100 2550 2300 2550
-Wire Wire Line
-	2100 2650 2300 2650
-Wire Wire Line
-	2150 3000 2150 2750
-Connection ~ 2150 2750
-Wire Wire Line
 	5350 5000 4850 5000
 $Comp
-L Earth #PWR1
+L Earth #PWR01
 U 1 1 5AB015D4
-P 2150 3000
-F 0 "#PWR1" H 2150 2750 50  0001 C CNN
-F 1 "Earth" H 2150 2850 50  0001 C CNN
-F 2 "" H 2150 3000 50  0001 C CNN
-F 3 "" H 2150 3000 50  0001 C CNN
-	1    2150 3000
+P 2050 3350
+F 0 "#PWR01" H 2050 3100 50  0001 C CNN
+F 1 "Earth" H 2050 3200 50  0001 C CNN
+F 2 "" H 2050 3350 50  0001 C CNN
+F 3 "" H 2050 3350 50  0001 C CNN
+	1    2050 3350
 	1    0    0    -1
 $EndComp
-Wire Wire Line
-	2150 2750 2100 2750
 Text Notes 3450 2550 0    60   ~ 0
 120V DC NOMINAL
@@
 	2250 4700 2500 4700
 Text Label 2250 4700 0    60   ~ 0
-3v3
+5v
 Text Label 3500 3600 0    60   ~ 0
-3v3
+5v
 Wire Wire Line
 	3500 3600 3350 3600
 $Comp
-L GNDD #PWR2
+L GNDD #PWR02
 U 1 1 5AB1DC44
 P 3650 5700
-F 0 "#PWR2" H 3650 5450 50  0001 C CNN
+F 0 "#PWR02" H 3650 5450 50  0001 C CNN
 F 1 "GNDD" H 3650 5575 50  0000 C CNN
 F 2 "" H 3650 5700 50  0001 C CNN
@@
 	7050 5000 7050 5100
 $Comp
-L GNDPWR #PWR3
+L GNDPWR #PWR03
 U 1 1 5AB1E9D9
 P 6850 5750
-F 0 "#PWR3" H 6850 5550 50  0001 C CNN
+F 0 "#PWR03" H 6850 5550 50  0001 C CNN
 F 1 "GNDPWR" H 6850 5620 50  0000 C CNN
 F 2 "" H 6850 5700 50  0001 C CNN
@@
 	6350 5000 7050 5000
 Text Label 3650 4850 0    60   ~ 0
-3v3
+5v
 Wire Wire Line
 	3650 4850 3850 4850
@@
 F7 "logic_pwr" I L 3850 4850 60
 $EndSheet
+Text Label 5200 5300 0    60   ~ 0
+5v
+Wire Wire Line
+	5200 5300 5350 5300
+Text Notes 1400 2150 0    60   ~ 0
+external voltage boost xformer may be applied for high voltage stage
+Text Notes 5200 2350 0    60   ~ 0
+check for dumb shit w/ pwr, gnd. don't kill people
+Text Notes 6700 4750 0    60   ~ 0
+coax sheath is connected to case gnd
+Text Notes 3500 3050 0    60   ~ 0
+substantially reduces board space if large reactifier off board
+Wire Wire Line
+	1950 2550 2300 2550
+Wire Wire Line
+	1950 2650 2300 2650
+Wire Wire Line
+	1950 2750 2300 2750
+Wire Wire Line
+	1950 2850 2300 2850
+Wire Wire Line
+	2050 3350 2050 2950
+Wire Wire Line
+	2050 2950 1950 2950
+Text Notes 1400 2300 0    60   ~ 0
+reactification for 240 supply is off board.
 $EndSCHEMATC
