File: Power_US_Driver/power_amp.sch (KiCad schematic (older format))
At the start: 9 parts, among them Q1 Q_NMOS_DGS, Q2 Q_NMOS_DGS, U2 IR2110

Commit message: moved high current diode off board
Parts:
- added Q3, Q4: IRF640N, TO_SOT_Packages_THT:TO-220-3_Vertical, symbol Q_NMOS_GDS
- Q1, Q2: value Q_NMOS_DGS -> MTH30N20; footprint (none) -> TO_SOT_Packages_THT:TO-218_SOT93_Vertical; symbol Q_NMOS_DGS -> Q_NMOS_GDS
Connections:
- net GNDPWR: now also Q4.3 (S)
- net US_POWER_OUT: now also Q2.2 (D), Q3.3 (S), Q4.2 (D); no longer Q2.1 (D)
- net v+: now also Q1.2 (D), Q3.2 (D); no longer Q1.1 (D)
- net at R3.1: now also Q1.1 (G), Q3.1 (G); no longer Q1.2 (G)
- net at R4.2: now also Q2.1 (G); no longer Q2.2 (G)
Other:
- note added: "DNI - INSTALL ONLY ONE"
- note added: "parrallel for TO220 and TO247 options"
- note removed: "VCC - low side supply. GNDPWR?"
- note removed: "check that -60 is ok"
- note removed: "has to be dragged to V- to turn off..."
- note removed: "two of these and an optoisolator?"
Changed lines of the file:
@@
 HEATSINKING IS CRITICAL FOR THIS COMPONENT
 $Comp
-L Q_NMOS_DGS Q1
+L Q_NMOS_GDS Q1
 U 1 1 5AAE8010
 P 6150 3600
 F 0 "Q1" H 6350 3650 50  0000 L CNN
-F 1 "Q_NMOS_DGS" H 6350 3550 50  0000 L CNN
-F 2 "" H 6350 3700 50  0001 C CNN
+F 1 "MTH30N20" H 6350 3550 50  0000 L CNN
+F 2 "TO_SOT_Packages_THT:TO-218_SOT93_Vertical" H 6350 3700 50  0001 C CNN
 F 3 "" H 6150 3600 50  0001 C CNN
 	1    6150 3600
 	1    0    0    -1
 $EndComp
-Text Notes 6500 3600 0    60   ~ 0
+Text Notes 6400 3350 0    60   ~ 0
 check pinout
 $Comp
@@
 INPUT THRESHOLDS, LOGIC SUPPLIES
 $Comp
-L GNDPWR #PWR13
+L GNDPWR #PWR012
 U 1 1 5AB00C48
 P 6250 4750
-F 0 "#PWR13" H 6250 4550 50  0001 C CNN
+F 0 "#PWR012" H 6250 4550 50  0001 C CNN
 F 1 "GNDPWR" H 6250 4620 50  0000 C CNN
 F 2 "" H 6250 4700 50  0001 C CNN
@@
 $EndComp
 $Comp
-L GNDD #PWR12
+L GNDD #PWR013
 U 1 1 5AB1B5F8
 P 4000 4100
-F 0 "#PWR12" H 4000 3850 50  0001 C CNN
+F 0 "#PWR013" H 4000 3850 50  0001 C CNN
 F 1 "GNDD" H 4000 3975 50  0000 C CNN
 F 2 "" H 4000 4100 50  0001 C CNN
@@
 Wire Wire Line
 	3150 3700 4300 3700
-Text Notes 3500 4700 0    60   ~ 0
-VCC - low side supply. GNDPWR?
 $Comp
 L C C8
@@
 $EndComp
 $Comp
-L GNDD #PWR11
+L GNDD #PWR014
 U 1 1 5AB1BA1D
 P 4000 3450
-F 0 "#PWR11" H 4000 3200 50  0001 C CNN
+F 0 "#PWR014" H 4000 3200 50  0001 C CNN
 F 1 "GNDD" H 4000 3325 50  0000 C CNN
 F 2 "" H 4000 3450 50  0001 C CNN
@@
 Connection ~ 3450 3700
 Connection ~ 5550 4750
-Text Notes 3550 4850 0    60   ~ 0
-check that -60 is ok
 Text Notes 5200 3200 0    60   ~ 0
 C, R values
 $Comp
-L Q_NMOS_DGS Q2
+L Q_NMOS_GDS Q2
 U 1 1 5AAE8077
 P 6150 4150
 F 0 "Q2" H 6350 4200 50  0000 L CNN
-F 1 "Q_NMOS_DGS" H 6350 4100 50  0000 L CNN
-F 2 "" H 6350 4250 50  0001 C CNN
+F 1 "MTH30N20" H 6350 4100 50  0000 L CNN
+F 2 "TO_SOT_Packages_THT:TO-218_SOT93_Vertical" H 6350 4250 50  0001 C CNN
 F 3 "" H 6150 4150 50  0001 C CNN
 	1    6150 4150
@@
 $EndComp
 Connection ~ 6000 4750
-Text Notes 6950 4150 0    60   ~ 0
-has to be dragged to V- to turn off...
-Text Notes 3900 5250 0    60   ~ 0
-two of these and an optoisolator?
 Wire Wire Line
 	5150 4200 5150 4450
@@
 	5950 4450 5950 4150
 Wire Wire Line
-	5250 4750 6250 4750
+	5250 4750 7050 4750
+Text Notes 6400 3250 0    60   ~ 0
+parrallel for TO220 and TO247 options
+Connection ~ 7050 3800
+Wire Wire Line
+	7050 3400 6250 3400
+Wire Wire Line
+	5950 3600 6750 3600
+Text Notes 7350 3450 0    60   ~ 0
+DNI - INSTALL ONLY ONE
+$Comp
+L Q_NMOS_GDS Q3
+U 1 1 5AB2E488
+P 6950 3600
+F 0 "Q3" H 7150 3650 50  0000 L CNN
+F 1 "IRF640N" H 7150 3550 50  0000 L CNN
+F 2 "TO_SOT_Packages_THT:TO-220-3_Vertical" H 7150 3700 50  0001 C CNN
+F 3 "" H 6950 3600 50  0001 C CNN
+	1    6950 3600
+	1    0    0    -1
+$EndComp
+$Comp
+L Q_NMOS_GDS Q4
+U 1 1 5AB2E4C8
+P 6950 4150
+F 0 "Q4" H 7150 4200 50  0000 L CNN
+F 1 "IRF640N" H 7150 4100 50  0000 L CNN
+F 2 "TO_SOT_Packages_THT:TO-220-3_Vertical" H 7150 4250 50  0001 C CNN
+F 3 "" H 6950 4150 50  0001 C CNN
+	1    6950 4150
+	1    0    0    -1
+$EndComp
+Wire Wire Line
+	7050 3950 7050 3800
+Wire Wire Line
+	7050 4750 7050 4350
+Connection ~ 6250 4750
+Wire Wire Line
+	6000 4150 6000 4500
+Wire Wire Line
+	6000 4500 6750 4500
+Wire Wire Line
+	6750 4500 6750 4150
+Text Notes 7350 4100 0    60   ~ 0
+DNI - INSTALL ONLY ONE
 $EndSCHEMATC
